File: xtremekeyboard1.kicad_sch (KiCad schematic)
At the start: 89 parts, among them J2 Conn_01x05_Pin, J3 Conn_01x05_Socket, J4 OLED-128x32, SW1 1u MX, SW10 1u MX, SW11 1u MX, SW12 1u MX, SW13 1u MX, SW14 1u MX, SW15 1u MX, SW16 1u MX, SW17 1u MX, SW18 1u MX, SW19 1u MX, SW2 1u MX, SW20 1u MX, SW21 1u MX, SW22 1u MX, SW23 1u MX, SW24 1u MX, SW25 1u MX, SW26 1u MX, SW27 1u MX, SW3 1u MX, SW4 1u MX, SW5 1u MX, SW6 1u MX, SW7 1u MX, SW8 1u MX, SW9 1u MX, U1 rp2040-zero, U2 PS4 Joystick

Commit message: finished PCB i think
Parts:
- renumbered SW1 to SW0,0, SW2 to SW0,1, SW3 to SW0,2, SW4 to SW0,3, SW5 to SW0,4, SW6 to SW0,5, SW7 to SW1,0, SW8 to SW1,1, SW9 to SW1,2, SW10 to SW1,3, SW11 to SW1,4, SW12 to SW1,5, SW13 to SW2,0, SW14 to SW2,1, SW15 to SW2,2, SW16 to SW2,3, SW17 to SW2,4, SW18 to SW2,5, SW19 to SW3,0, SW20 to SW3,1, SW21 to SW3,2, SW22 to SW3,3, SW23 to SW3,4, SW24 to SW3,5, SW25 to SW4,3, SW26 to SW4,4, SW27 to SW4,5
Changed lines of the file:
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@@
 		(on_board yes)
 		(dnp no)
-		(property "Reference" "SW4"
+		(property "Reference" "SW0,3"
 			(at 67.31 48.26 0)
 			(effects
@@
 			(project "xtremekeyboard1"
 				(path "/984cae9b-27c7-49b6-85c2-c1b90de6856e"
-					(reference "SW4")
+					(reference "SW0,3")
 					(unit 1)
 				)
@@
 		(on_board yes)
 		(dnp no)
-		(property "Reference" "SW24"
+		(property "Reference" "SW3,5"
 			(at 85.09 97.79 0)
 			(effects
@@
 			(project "xtremekeyboard1"
 				(path "/984cae9b-27c7-49b6-85c2-c1b90de6856e"
-					(reference "SW24")
+					(reference "SW3,5")
 					(unit 1)
 				)
@@
 		(on_board yes)
 		(dnp no)
-		(property "Reference" "SW15"
+		(property "Reference" "SW2,2"
 			(at 58.42 81.28 0)
 			(effects
@@
 			(project "xtremekeyboard1"
 				(path "/984cae9b-27c7-49b6-85c2-c1b90de6856e"
-					(reference "SW15")
+					(reference "SW2,2")
 					(unit 1)
 				)
@@
 		(on_board yes)
 		(dnp no)
-		(property "Reference" "SW22"
+		(property "Reference" "SW3,3"
 			(at 67.31 97.79 0)
 			(effects
@@
 			(project "xtremekeyboard1"
 				(path "/984cae9b-27c7-49b6-85c2-c1b90de6856e"
-					(reference "SW22")
+					(reference "SW3,3")
 					(unit 1)
 				)
@@
 		(on_board yes)
 		(dnp no)
-		(property "Reference" "SW14"
+		(property "Reference" "SW2,1"
 			(at 49.53 81.28 0)
 			(effects
@@
 			(project "xtremekeyboard1"
 				(path "/984cae9b-27c7-49b6-85c2-c1b90de6856e"
-					(reference "SW14")
+					(reference "SW2,1")
 					(unit 1)
 				)
@@
 		(on_board yes)
 		(dnp no)
-		(property "Reference" "SW2"
+		(property "Reference" "SW0,1"
 			(at 49.53 48.26 0)
 			(effects
@@
 			(project "xtremekeyboard1"
 				(path "/984cae9b-27c7-49b6-85c2-c1b90de6856e"
-					(reference "SW2")
+					(reference "SW0,1")
 					(unit 1)
 				)
@@
 		(on_board yes)
 		(dnp no)
-		(property "Reference" "SW1"
+		(property "Reference" "SW0,0"
 			(at 40.64 48.26 0)
 			(effects
@@
 			(project "xtremekeyboard1"
 				(path "/984cae9b-27c7-49b6-85c2-c1b90de6856e"
-					(reference "SW1")
+					(reference "SW0,0")
 					(unit 1)
 				)
@@
 		(on_board yes)
 		(dnp no)
-		(property "Reference" "SW26"
+		(property "Reference" "SW4,4"
 			(at 76.2 114.3 0)
 			(effects
@@
 			(project "xtremekeyboard1"
 				(path "/984cae9b-27c7-49b6-85c2-c1b90de6856e"
-					(reference "SW26")
+					(reference "SW4,4")
 					(unit 1)
 				)
@@
 		(on_board yes)
 		(dnp no)
-		(property "Reference" "SW10"
+		(property "Reference" "SW1,3"
 			(at 67.31 64.77 0)
 			(effects
@@
 			(project "xtremekeyboard1"
 				(path "/984cae9b-27c7-49b6-85c2-c1b90de6856e"
-					(reference "SW10")
+					(reference "SW1,3")
 					(unit 1)
 				)
@@
 		(on_board yes)
 		(dnp no)
-		(property "Reference" "SW16"
+		(property "Reference" "SW2,3"
 			(at 67.31 81.28 0)
 			(effects
@@
 			(project "xtremekeyboard1"
 				(path "/984cae9b-27c7-49b6-85c2-c1b90de6856e"
-					(reference "SW16")
+					(reference "SW2,3")
 					(unit 1)
 				)
@@
 		(on_board yes)
 		(dnp no)
-		(property "Reference" "SW23"
+		(property "Reference" "SW3,4"
 			(at 76.2 97.79 0)
 			(effects
@@
 			(project "xtremekeyboard1"
 				(path "/984cae9b-27c7-49b6-85c2-c1b90de6856e"
-					(reference "SW23")
+					(reference "SW3,4")
 					(unit 1)
 				)
@@
 		(on_board yes)
 		(dnp no)
-		(property "Reference" "SW17"
+		(property "Reference" "SW2,4"
 			(at 76.2 81.28 0)
 			(effects
@@
 			(project "xtremekeyboard1"
 				(path "/984cae9b-27c7-49b6-85c2-c1b90de6856e"
-					(reference "SW17")
+					(reference "SW2,4")
 					(unit 1)
 				)
@@
 		(on_board yes)
 		(dnp no)
-		(property "Reference" "SW12"
+		(property "Reference" "SW1,5"
 			(at 85.09 64.77 0)
 			(effects
@@
 			(project "xtremekeyboard1"
 				(path "/984cae9b-27c7-49b6-85c2-c1b90de6856e"
-					(reference "SW12")
+					(reference "SW1,5")
 					(unit 1)
 				)
@@
 		(on_board yes)
 		(dnp no)
-		(property "Reference" "SW9"
+		(property "Reference" "SW1,2"
 			(at 58.42 64.77 0)
 			(effects
@@
 			(project "xtremekeyboard1"
 				(path "/984cae9b-27c7-49b6-85c2-c1b90de6856e"
-					(reference "SW9")
+					(reference "SW1,2")
 					(unit 1)
 				)
@@
 		(on_board yes)
 		(dnp no)
-		(property "Reference" "SW3"
+		(property "Reference" "SW0,2"
 			(at 58.42 48.26 0)
 			(effects
@@
 			(project "xtremekeyboard1"
 				(path "/984cae9b-27c7-49b6-85c2-c1b90de6856e"
-					(reference "SW3")
+					(reference "SW0,2")
 					(unit 1)
 				)
@@
 		(on_board yes)
 		(dnp no)
-		(property "Reference" "SW6"
+		(property "Reference" "SW0,5"
 			(at 85.09 48.26 0)
 			(effects
@@
 			(project "xtremekeyboard1"
 				(path "/984cae9b-27c7-49b6-85c2-c1b90de6856e"
-					(reference "SW6")
+					(reference "SW0,5")
 					(unit 1)
 				)
@@
 		(on_board yes)
 		(dnp no)
-		(property "Reference" "SW7"
+		(property "Reference" "SW1,0"
 			(at 40.64 64.77 0)
 			(effects
@@
 			(project "xtremekeyboard1"
 				(path "/984cae9b-27c7-49b6-85c2-c1b90de6856e"
-					(reference "SW7")
+					(reference "SW1,0")
 					(unit 1)
 				)
@@
 		(on_board yes)
 		(dnp no)
-		(property "Reference" "SW25"
+		(property "Reference" "SW4,3"
 			(at 67.31 114.3 0)
 			(effects
@@
 			(project "xtremekeyboard1"
 				(path "/984cae9b-27c7-49b6-85c2-c1b90de6856e"
-					(reference "SW25")
+					(reference "SW4,3")
 					(unit 1)
 				)
@@
 		(on_board yes)
 		(dnp no)
-		(property "Reference" "SW8"
+		(property "Reference" "SW1,1"
 			(at 49.53 64.77 0)
 			(effects
@@
 			(project "xtremekeyboard1"
 				(path "/984cae9b-27c7-49b6-85c2-c1b90de6856e"
-					(reference "SW8")
+					(reference "SW1,1")
 					(unit 1)
 				)
@@
 		(on_board yes)
 		(dnp no)
-		(property "Reference" "SW18"
+		(property "Reference" "SW2,5"
 			(at 85.09 81.28 0)
 			(effects
@@
 			(project "xtremekeyboard1"
 				(path "/984cae9b-27c7-49b6-85c2-c1b90de6856e"
-					(reference "SW18")
+					(reference "SW2,5")
 					(unit 1)
 				)
@@
 		(on_board yes)
 		(dnp no)
-		(property "Reference" "SW20"
+		(property "Reference" "SW3,1"
 			(at 49.53 97.79 0)
 			(effects
@@
 			(project "xtremekeyboard1"
 				(path "/984cae9b-27c7-49b6-85c2-c1b90de6856e"
-					(reference "SW20")
+					(reference "SW3,1")
 					(unit 1)
 				)
@@
 		(on_board yes)
 		(dnp no)
-		(property "Reference" "SW13"
+		(property "Reference" "SW2,0"
 			(at 40.64 81.28 0)
 			(effects
@@
 			(project "xtremekeyboard1"
 				(path "/984cae9b-27c7-49b6-85c2-c1b90de6856e"
-					(reference "SW13")
+					(reference "SW2,0")
 					(unit 1)
 				)
@@
 		(on_board yes)
 		(dnp no)
-		(property "Reference" "SW11"
+		(property "Reference" "SW1,4"
 			(at 76.2 64.77 0)
 			(effects
@@
 			(project "xtremekeyboard1"
 				(path "/984cae9b-27c7-49b6-85c2-c1b90de6856e"
-					(reference "SW11")
+					(reference "SW1,4")
 					(unit 1)
 				)
@@
 		(on_board yes)
 		(dnp no)
-		(property "Reference" "SW5"
+		(property "Reference" "SW0,4"
 			(at 76.2 48.26 0)
 			(effects
@@
 			(project "xtremekeyboard1"
 				(path "/984cae9b-27c7-49b6-85c2-c1b90de6856e"
-					(reference "SW5")
+					(reference "SW0,4")
 					(unit 1)
 				)
@@
 		(on_board yes)
 		(dnp no)
-		(property "Reference" "SW19"
+		(property "Reference" "SW3,0"
 			(at 40.64 97.79 0)
 			(effects
@@
 			(project "xtremekeyboard1"
 				(path "/984cae9b-27c7-49b6-85c2-c1b90de6856e"
-					(reference "SW19")
+					(reference "SW3,0")
 					(unit 1)
 				)
@@
 		(on_board yes)
 		(dnp no)
-		(property "Reference" "SW27"
+		(property "Reference" "SW4,5"
 			(at 85.09 114.3 0)
 			(effects
@@
 			(project "xtremekeyboard1"
 				(path "/984cae9b-27c7-49b6-85c2-c1b90de6856e"
-					(reference "SW27")
+					(reference "SW4,5")
 					(unit 1)
 				)
@@
 		(on_board yes)
 		(dnp no)
-		(property "Reference" "SW21"
+		(property "Reference" "SW3,2"
 			(at 58.42 97.79 0)
 			(effects
@@
 			(project "xtremekeyboard1"
 				(path "/984cae9b-27c7-49b6-85c2-c1b90de6856e"
-					(reference "SW21")
+					(reference "SW3,2")
 					(unit 1)
 				)
